File: pcb_central_unit/RBY_tireuse.sch (KiCad schematic (older format))
At the start: 9 parts, among them J1 CMD_PAN, J2 GLASS_0, J3 GLASS_1, J4 Conn_01x04_Female, J5 Conn_01x04_Female, J6 DCDC_BOOSTER, J7 Conn_01x02_Male, U2 TMC2208_SILENTSTEPSTICK, U3 TMC2208_SILENTSTEPSTICK

Commit message: PCB V2
Parts:
- removed U2, U3: TMC2208_SILENTSTEPSTICK, MODULE_ESP32:MODULE_TMC2208_SILENTSTEPSTICK, symbol TMC2208_SILENTSTEPSTICK:TMC2208_SILENTSTEPSTICK
- added J8: SPARE_GPIO_0, Connector_PinHeader_2.54mm:PinHeader_1x02_P2.54mm_Horizontal, symbol Connector:Conn_01x02_Male
- added J9: SPARE_GPIO_1, Connector_PinHeader_2.54mm:PinHeader_1x02_P2.54mm_Horizontal, symbol Connector:Conn_01x02_Male
- added R1, R2: 1kOHM, Resistor_THT:R_Axial_DIN0207_L6.3mm_D2.5mm_P7.62mm_Horizontal, symbol Device:R
- added U1, U2: TMC2208_SILENTSTEPSTICK-TMC2208_SILENTSTEPSTICK, ProjectModules:MODULE_TMC2208_SILENTSTEPSTICK, symbol MODULES:TMC2208_SILENTSTEPSTICK-TMC2208_SILENTSTEPSTICK
- added U3: ESP32_DevKit_V1_DOIT_30_pin, ProjectModules:esp32_devkit_v1_doit, symbol MODULES:ESP32_DevKit_V1_DOIT_30_pin
- J4: value Conn_01x04_Female -> STEPPER_0
- J5: value Conn_01x04_Female -> STEPPER_1
- J6: footprint Connector_PinHeader_2.54mm:PinHeader_1x04_P2.54mm_Horizontal -> Connector_PinHeader_2.54mm:PinHeader_1x04_P2.54mm_Vertical
- J7: value Conn_01x02_Male -> ALIM_5V; footprint Connector_PinHeader_2.54mm:PinHeader_1x02_P2.54mm_Horizontal -> Connector_PinHeader_2.54mm:PinHeader_1x02_P2.54mm_Vertical
Connections:
- net labels added: UART_0, UART_1
- wire segments 80 -> 109
Other:
- moved on the sheet: J6, J7
